Commit message: update urdf mesh

File: urdf/xacros/psen_scan.urdf.xacro (robot description, xacro)
@@ -5,5 +5,5 @@
     <xacro:property name="radius" value="0.051" /> <!-- src datasheet p 96 -->
     <xacro:property name="height" value="0.152" /> <!-- src datasheet p 96 -->
-    <xacro:property name="dist_scanning_plane_top" value="0.0377" /> <!-- src datasheet p 96 -->
+    <xacro:property name="dist_scanning_plane_top" value="0.02" /> <!-- src datasheet p 96 -->
     <xacro:property name="dist_scanning_axis_rear" value="0.0525" /> <!-- src datasheet p 96 -->
     <joint name="${prefix}_joint" type="fixed">
@@ -22,7 +22,7 @@
     <link name="${prefix}_body_link">
       <visual>
-        <origin xyz="-0.016 0 -0.039" rpy="0 0 3.14" />
+        <origin xyz="${-radius} 0 0" rpy="1.57 0 0" />
         <geometry>
-          <mesh filename="package://psen_scan_v2/urdf/meshes/PSENscan.dae" scale="0.001 0.001 0.001"/>
+          <mesh filename="package://psen_scan_v2/urdf/meshes/psenscan.glb" scale="1 1 1"/>
         </geometry>
         <material name="pilz_yellow" >
@@ -31,7 +31,7 @@
       </visual>
       <collision>
-        <origin xyz="-0.016 0 -0.039" rpy="0 0 3.14" />
+        <origin xyz="${-radius} 0 0" rpy="1.57 0 0" />
         <geometry>
-          <mesh filename="package://psen_scan_v2/urdf/meshes/PSENscan.dae" scale="0.001 0.001 0.001"/>
+          <mesh filename="package://psen_scan_v2/urdf/meshes/psenscan.glb" scale="1 1 1"/>
         </geometry>
       </collision>
@@ -47,5 +47,5 @@
       <parent link="${prefix}_body_link" />
       <child link="${prefix}" />
-      <origin rpy="${pi} 0 0" xyz="0 ${radius - dist_scanning_axis_rear} ${height / 2 - dist_scanning_plane_top}"/>
+      <origin rpy="3.14 0 0" xyz="0 ${radius - dist_scanning_axis_rear} ${height / 2 - dist_scanning_plane_top}"/>
     </joint>
     <!-- This is the location of the laser scan -->
